File: customESP32board/customESP32board.kicad_pcb (KiCad board)
At the start: 2 copper layers, 60 x 60 mm, 47 parts, among them J1 USB_B_Micro, J2 Conn_01x16_Pin, J3 Conn_01x16_Pin, Q1 S8050, Q2 S8050, Q3 BSS138, Q4 BSS138, Q5 BSS138, SW1 SW_Push, SW2 SW_Push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

Commit message: updates
Parts:
- moved D6 7.28 mm to (162.3, 104.1)
- moved D7 7.28 mm to (162.3, 110.8)
- moved R7 7.28 mm to (162.5, 99.1)
- moved R8 7.28 mm to (160.0, 99.1)
- moved R9 7.28 mm to (157.5, 99.1)
- moved D8 7.27 mm to (162.5, 117.5)
- moved R15 0.50 mm to (111.0, 106.7)
- moved R18 0.50 mm to (108.5, 106.7)
- moved R14 0.35 mm to (113.8, 100.8)
- moved R17 0.35 mm to (111.2, 100.8)
- moved R16 0.25 mm to (116.2, 100.5)
Routing:
- net +5V: track 0.00 -> 53.6 mm
- net ESP_IO27: track 0.00 -> 24.2 mm
- net ESP_IO21: track 0.00 -> 23.8 mm
- net ESP_IO26: track 0.00 -> 20.9 mm
- net ESP_IO19: track 0.00 -> 18.8 mm
- net RGB_RED: track 0.00 -> 18.1 mm
- net RGB_GREEN: track 0.00 -> 18.1 mm
- net RGB_BLUE: track 0.00 -> 17.8 mm
- net ESP_IO0: track 0.00 -> 15.4 mm
- net ESP_IO18: track 0.00 -> 14.9 mm
- net ESP_IO4: track 0.00 -> 14.8 mm
- net ESP_IO12: track 0.00 -> 14.3 mm
- net ESP_IO14: track 0.00 -> 13.7 mm
- net ESP_IO16: track 0.00 -> 13.5 mm
- net ESP_IO25: track 0.00 -> 13.0 mm
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